File: Eagle/Agrovoltaic/Board.sch (EAGLE design)
At the start: 78 parts, among them J1 WAGO-03BE, J2 WAGO-03BE, J3 WAGO-03BE, K1 SRD-05VDC-SL-C, K3 SRD-05VDC-SL-C, Q1 BC338, Q2 BC338, U2 DEVKIT_V1_ESP32-WROOM-32

Commit message: EDIT:Mengedit Board
Parts:
- renumbered C5 to CA1, C6 to CA2, D15 to DZA2, D16 to DZA4, D17 to DZA1, D18 to DZA3, R21 to RA11, R22 to RA12, R27 to RA13, R28 to RA21, R29 to RA22, R30 to RA23, X4 to XOUTPUT, X5 to XINPUT
Connections:
- net OUT1+: now also XOUTPUT-1.KL; no longer XOUTPUT-4.KL
- net OUT2+: now also XOUTPUT-2.KL; no longer XOUTPUT-3.KL
- net OUT3+: now also XOUTPUT-3.KL; no longer XOUTPUT-2.KL
- net OUT4+: now also XOUTPUT-4.KL; no longer XOUTPUT-1.KL
